Commit message: add many packages

File: xiaoqiang_description/robots/xiaoqiang_urdf.URDF (robot description, URDF)
Before this commit: robot xiaoqiang_udrf, 6 links, 5 joints
Links:
- link back_wheel: geometry collision mesh filename=package://xiaoqiang_description/meshes/back_wheel.STL; visual mesh filename=package://xiaoqiang_description/meshes/back_wheel.STL
- link base_link: geometry collision mesh filename=package://xiaoqiang_description/meshes/base_link.STL; visual mesh filename=package://xiaoqiang_description/meshes/base_link.STL
- link kinect_Link: geometry collision mesh filename=package://xiaoqiang_description/meshes/kinect_Link.STL; visual mesh filename=package://xiaoqiang_description/meshes/kinect_Link.STL
- link left_wheel: geometry collision mesh filename=package://xiaoqiang_description/meshes/left_wheel.STL; visual mesh filename=package://xiaoqiang_description/meshes/left_wheel.STL
- link lidar_link: geometry collision mesh filename=package://xiaoqiang_description/meshes/lidar_link.STL; visual mesh filename=package://xiaoqiang_description/meshes/lidar_link.STL
- link right_wheel: geometry collision mesh filename=package://xiaoqiang_description/meshes/right_wheel.STL; visual mesh filename=package://xiaoqiang_description/meshes/right_wheel.STL
